File: pcb/ohmmeter/ohmmeter.kicad_pcb (KiCad board)
At the start: 2 copper layers, 82.4 x 92.3 mm, 37 parts, among them J1 DUT, J2 DUT, J3 ISP, J4 DUT, SW1 SW_Push, U1 ATMEGA88PA-MU, U2 MCP1640BCH, U3 TP4056

Commit message: PCB update
fixed silk
Other:
- board text added: "Ohmmeter nach Zabex & Axel S. 2020"
- board text removed: "Ohmmeter nach Zabex & Alex S. 2020"
